File: so_101_demo_board/mainBoard.kicad_sch (KiCad schematic)
At the start: 60 parts, among them J1 XT60PW-M, J2 XT60PW-M, J21 B2B-PH_K, J22 Conn_01x02, J3 XT30PW-M, J4 XT30PW-M, Q1 FQD11P06TM, Q2 FQD11P06TM, U1 TPS565208, U2 TPS565208

Commit message: did some updating to mainboard, added a demo board
Parts:
- added C19, C7: 10uF, Capacitor_SMD:C_0805_2012Metric_Pad1.18x1.45mm_HandSolder, symbol Device:C
- added C20, C21: 0.1uF, Capacitor_SMD:C_0805_2012Metric_Pad1.18x1.45mm_HandSolder, symbol Device:C
- added C22, C23, C25: 22uF, Capacitor_SMD:C_0805_2012Metric_Pad1.18x1.45mm_HandSolder, symbol Device:C
- added D4: LED, Diode_SMD:D_0805_2012Metric_Pad1.15x1.40mm_HandSolder, symbol Device:LED
- added J17, J5: 2 pin screw, TerminalBlock_Phoenix:TerminalBlock_Phoenix_MKDS-1,5-2_1x02_P5.00mm_Horizontal, symbol Connector:Screw_Terminal_01x02
- added L5: 3.3uH, Inductor_SMD:L_Abracon_ASPI-0630LR, symbol Device:L_Ferrite
- added Q3: FQD11P06TM, Package_TO_SOT_SMD:TO-252-2, symbol FQD11P06TM:FQD11P06TM
- added R23: 0, Resistor_SMD:R_1210_3225Metric_Pad1.30x2.65mm_HandSolder, symbol Device:R_US
- added R27: 100, Resistor_SMD:R_0805_2012Metric_Pad1.20x1.40mm_HandSolder, symbol Device:R_US
- added R28, R29: 10K, Resistor_SMD:R_0805_2012Metric_Pad1.20x1.40mm_HandSolder, symbol Device:R_US
- added R30: 87370, Resistor_SMD:R_0805_2012Metric_Pad1.20x1.40mm_HandSolder, symbol Device:R_US
- added R31: 1K, Resistor_SMD:R_0805_2012Metric_Pad1.20x1.40mm_HandSolder, symbol Device:R_US
- added TP3: TestPoint_Probe, TestPoint:TestPoint_Pad_D2.0mm, symbol Connector:TestPoint_Probe
- added U3: TPS565208, Package_TO_SOT_SMD:SOT-23-6, symbol Regulator_Switching:TPS565208
- R4, R5: value 1k -> 500
- R8: value 1k -> 300
Connections:
- net +12V: now also Q3.3 (D), R23.2, R28.1
- net GND: now also C19.2, C20.2, C22.2, C23.2, C25.2, C7.2, D4.1 (K), J17.2 (Pin_2), J5.2 (Pin_2), R27.2, R29.1, U3.1 (GND)
- new net: C19.1, C20.1, C7.1, Q3.2 (S), R23.1, U3.3 (VIN)
- new net: C21.1, U3.6 (VBST)
- new net: C21.2, L5.1, U3.2 (SW)
- new net: R29.2, R30.1, U3.4 (VFB)
- new net: R28.2, U3.5 (EN)
- new net: Q3.1 (G), R27.1
- new net: D4.2 (A), R31.2
- new net 7.4V: C22.1, C23.1, C25.1, J17.1 (Pin_1), J5.1 (Pin_1), L5.2, R30.2, R31.1, TP3.1
Other:
- note added: "12V to 7.4V, 5A"
- note added: "For Servos"
