File: 25-26_NEW_mecanumDriveTrain/NEW_mecanumDriveTrain_25-26.kicad_pcb (KiCad board)
At the start: 2 copper layers, 174.3 x 85.8 mm, 39 parts, among them J1 JST-PH-K, J2 XT-30, J3 5 pin dupont, J4 5 pin dupont, J5 5 pin dupont, J6 5 pin dupont, U1 Teensy4.1, U2 PTCAN3414DR, U3 LD1117S50TR_SOT223, U4 Pololu 18v17 Motor Driver, U5 Pololu 18v17 Motor Driver, U6 Pololu 18v17 Motor Driver, U7 Pololu 18v17 Motor Driver

Commit message: did a review
Routing:
- net C_TX: track 64.3 -> 65.6 mm
- net GND: vias 178 -> 264

Commit message: Finished up mecanum board
Parts:
- added D1: CUHS20S60,H3F, Diode_SMD:D_SOD-323_HandSoldering, F.Cu at (149.4, 72.4)
- moved C2 3.19 mm to (137.4, 70.5)
- moved R1 2.62 mm to (141.3, 70.5)
- moved C4 2.34 mm to (150.6, 75.4)
- moved U2 1.98 mm to (143.0, 77.5)
- moved R2 0.68 mm to (145.0, 70.5), turned to 180 degrees
Connections:
- C4 pad 2: VCC -> Net-(D1-K)
- U3 pad 3: VCC -> Net-(D1-K)
Routing:
- net VCC: track 50.5 -> 45.2 mm
- net Net-(C2-Pad2): track 6.49 -> 10.6 mm, vias 0 -> 2
- net Net-(D1-K): track 0.00 -> 3.94 mm
- net +3.3V: track 288.2 -> 292.1 mm
- net C_RX: track 65.1 -> 63.5 mm
- net C_TX: track 65.6 -> 64.1 mm
- net CANN: track 9.61 -> 10.8 mm
- net CANP: track 9.98 -> 10.8 mm
- net GND: vias 264 -> 263
- net +12V: vias 28 -> 27
Other:
- board text added: "1"
- board text added: "3V3"
- board text added: "ENA"
- board text added: "ENB"
