File: 25-26_NEW_mecanumDriveTrain/NEW_mecanumDriveTrain_25-26.kicad_sch (KiCad schematic)
At the start: 38 parts, among them J1 JST-PH-K, J2 XT-30, J3 5 pin dupont, J4 5 pin dupont, J5 5 pin dupont, J6 5 pin dupont, U1 Teensy4.1, U2 PTCAN3414DR, U3 LD1117S50TR_SOT223, U4 Pololu 18v17 Motor Driver, U5 Pololu 18v17 Motor Driver, U6 Pololu 18v17 Motor Driver, U7 Pololu 18v17 Motor Driver

Commit message: Finished up mecanum board
Parts:
- added D1: CUHS20S60,H3F, Diode_SMD:D_SOD-323_HandSoldering, symbol Device:D_Schottky
Connections:
- net VCC: now also D1.2 (A); no longer C4.2, U3.3 (VI)
- new net: C4.2, D1.1 (K), U3.3 (VI)
Other:
- moved on the sheet: J2
Changed lines of the file:
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@@
 	)
 	(junction
-		(at 176.53 34.29)
+		(at 31.75 33.02)
 		(diameter 0)
 		(color 0 0 0 0)
 	)
 	(junction
-		(at 31.75 33.02)
+		(at 48.26 30.48)
 		(diameter 0)
 		(color 0 0 0 0)
 	)
 	(junction
-		(at 48.26 30.48)
+		(at 176.53 34.29)
 		(diameter 0)
 		(color 0 0 0 0)
@@
 	(wire
 		(pts
+			(xy 176.53 34.29) (xy 185.42 34.29)
+		)
+		(stroke
+			(width 0)
+			(type default)
+		)
+	)
+	(wire
+		(pts
 			(xy 59.69 35.56) (xy 52.07 35.56)
 		)
@@
 	(wire
 		(pts
+			(xy 193.04 34.29) (xy 195.58 34.29)
+		)
+		(stroke
+			(width 0)
+			(type default)
+		)
+	)
+	(wire
+		(pts
 			(xy 52.07 33.02) (xy 52.07 30.48)
 		)
@@
 	(symbol
 		(lib_id "power:VCC")
-		(at 176.53 34.29 270)
+		(at 195.58 34.29 270)
 		(unit 1)
 		(exclude_from_sim no)
@@
 		(fields_autoplaced yes)
 		(property "Reference" "#PWR09"
-			(at 172.72 34.29 0)
+			(at 191.77 34.29 0)
 			(effects
 				(font
@@
 		)
 		(property "Value" "VCC"
-			(at 180.34 34.2899 90)
+			(at 199.39 34.2899 90)
 			(effects
 				(font
@@
 		)
 		(property "Footprint" ""
-			(at 176.53 34.29 0)
+			(at 195.58 34.29 0)
 			(effects
 				(font
@@
 		)
 		(property "Datasheet" ""
-			(at 176.53 34.29 0)
+			(at 195.58 34.29 0)
 			(effects
 				(font
@@
 		)
 		(property "Description" "Power symbol creates a global label with name \"VCC\""
-			(at 176.53 34.29 0)
+			(at 195.58 34.29 0)
 			(effects
 				(font
@@
 	(symbol
 		(lib_id "Connector_Generic:Conn_01x02")
-		(at 203.2 31.75 0)
+		(at 203.2 24.13 0)
 		(unit 1)
 		(exclude_from_sim no)
@@
 		(fields_autoplaced yes)
 		(property "Reference" "J2"
-			(at 205.74 31.7499 0)
+			(at 205.74 24.1299 0)
 			(effects
 				(font
@@
 		)
 		(property "Value" "XT-30"
-			(at 205.74 34.2899 0)
+			(at 205.74 26.6699 0)
 			(effects
 				(font
@@
 		)
 		(property "Footprint" "Connector_AMASS:AMASS_XT30U-F_1x02_P5.0mm_Vertical"
-			(at 203.2 31.75 0)
+			(at 203.2 24.13 0)
 			(effects
 				(font
@@
 		)
 		(property "Datasheet" "~"
-			(at 203.2 31.75 0)
+			(at 203.2 24.13 0)
 			(effects
 				(font
@@
 		)
 		(property "Description" "Generic connector, single row, 01x02, script generated (kicad-library-utils/schlib/autogen/connector/)"
-			(at 203.2 31.75 0)
+			(at 203.2 24.13 0)
 			(effects
 				(font
@@
 	(symbol
 		(lib_id "power:GND")
-		(at 198.12 31.75 270)
+		(at 198.12 24.13 270)
 		(unit 1)
 		(exclude_from_sim no)
@@
 		(fields_autoplaced yes)
 		(property "Reference" "#PWR06"
-			(at 191.77 31.75 0)
+			(at 191.77 24.13 0)
 			(effects
 				(font
@@
 		)
 		(property "Value" "GND"
-			(at 194.31 31.7499 90)
+			(at 194.31 24.1299 90)
 			(effects
 				(font
@@
 		)
 		(property "Footprint" ""
-			(at 198.12 31.75 0)
+			(at 198.12 24.13 0)
 			(effects
 				(font
@@
 		)
 		(property "Datasheet" ""
-			(at 198.12 31.75 0)
+			(at 198.12 24.13 0)
 			(effects
 				(font
@@
 		)
 		(property "Description" "Power symbol creates a global label with name \"GND\" , ground"
-			(at 198.12 31.75 0)
+			(at 198.12 24.13 0)
 			(effects
 				(font
@@
 	(symbol
 		(lib_id "power:+12V")
-		(at 198.12 34.29 90)
+		(at 198.12 26.67 90)
 		(unit 1)
 		(exclude_from_sim no)
@@
 		(fields_autoplaced yes)
 		(property "Reference" "#PWR07"
-			(at 201.93 34.29 0)
+			(at 201.93 26.67 0)
 			(effects
 				(font
@@
 		)
 		(property "Value" "+12V"
-			(at 194.31 34.2899 90)
+			(at 194.31 26.6699 90)
 			(effects
 				(font
@@
 		)
 		(property "Footprint" ""
-			(at 198.12 34.29 0)
+			(at 198.12 26.67 0)
 			(effects
 				(font
@@
 		)
 		(property "Datasheet" ""
-			(at 198.12 34.29 0)
+			(at 198.12 26.67 0)
 			(effects
 				(font
@@
 		)
 		(property "Description" "Power symbol creates a global label with name \"+12V\""
-			(at 198.12 34.29 0)
+			(at 198.12 26.67 0)
 			(effects
 				(font
@@
 					(unit 1)
 				)
+			)
+		)
+	)
+	(symbol
+		(lib_id "Device:D_Schottky")
+		(at 189.23 34.29 0)
+		(unit 1)
+		(exclude_from_sim no)
+		(in_bom yes)
+		(on_board yes)
+		(dnp no)
+		(property "Reference" "D1"
+			(at 189.23 32.004 0)
+			(effects
+				(font
+					(size 1.27 1.27)
+				)
+			)
+		)
+		(property "Value" "CUHS20S60,H3F"
+			(at 189.23 36.83 0)
+			(effects
+				(font
+					(size 1.27 1.27)
+				)
+			)
+		)
+		(property "Footprint" "Diode_SMD:D_SOD-323_HandSoldering"
+			(at 189.23 34.29 0)
+			(effects
+				(font
+					(size 1.27 1.27)
+				)
+				(hide yes)
+			)
+		)
+		(property "Datasheet" "https://toshiba.semicon-storage.com/info/CUHS20S60_datasheet_en_20250926.pdf?did=70190&prodName=CUHS20S60"
+			(at 189.23 34.29 0)
+			(effects
+				(font
+					(size 1.27 1.27)
+				)
+				(hide yes)
+			)
+		)
+		(property "Description" "Schottky Diode"
+			(at 189.23 34.29 0)
+			(effects
+				(font
+					(size 1.27 1.27)
+				)
+				(hide yes)
+			)
+		)
+		(pin "2"
+		)
+		(pin "1"
+		)
+		(instances
+			(project ""
+				(path "/eb6ae2a8-b7b3-4c30-a8b9-bd96e5b62c41"
+					(reference "D1")
+					(unit 1)
+				)
