File: knob_board/knob_board.kicad_sch (KiCad schematic)
At the start: 36 parts, among them J1 xt30, J2 JST-PH-K, J3 Conn_01x03_Pin, J4 Conn_01x03_Pin, J5 Conn_01x03_Pin, J6 Conn_01x03_Pin, J7 Conn_01x03_Pin, Q1 BSS138, Q2 BSS138, Q3 BSS138, Q4 BSS138, Q5 BSS138, U1 Teensy4.1, U2 LD1117S50TR_SOT223, U3 PTCAN3414DDFR

Commit message: fixed minor issue, removed unecessary items
Parts:
- removed C2: 0.1uF, Capacitor_SMD:C_0805_2012Metric_Pad1.18x1.45mm_HandSolder, symbol Device:C
- removed U2: LD1117S50TR_SOT223, Package_TO_SOT_SMD:SOT-223-3_TabPin2, symbol Regulator_Linear:LD1117S50TR_SOT223
Other:
- moved on the sheet: C1
